File: hardware/DEBUGEDGE_BREAKOUT/DEBUGEDGE_BREAKOUT.kicad_sch (KiCad schematic)
At the start: 3 parts, among them J1 DebugEdge_02x05, J2 Conn_ARM_JTAG_SWD_10, J3 Conn_01x10_Pin

Commit message: Fix footprints and jlc placeholder in DebugEdge Breakout
Parts:
- J3: footprint Connector_PinSocket_2.54mm:PinSocket_1x10_P2.54mm_Vertical -> Connector_PinHeader_2.54mm:PinHeader_1x10_P2.54mm_Vertical
Changed lines of the file:
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@@
       (effects (font (size 1.27 1.27)) (justify right))
     )
-    (property "Footprint" "Connector_PinSocket_2.54mm:PinSocket_1x10_P2.54mm_Vertical" (at 141.605 100.965 0)
+    (property "Footprint" "Connector_PinHeader_2.54mm:PinHeader_1x10_P2.54mm_Vertical" (at 141.605 100.965 0)
       (effects (font (size 1.27 1.27)) hide)
     )
